File: kicad/modulo buck boost.kicad_pcb (KiCad board)
At the start: 2 copper layers, 54.4 x 25.6 mm, 16 parts, among them J1 USB_B_Micro, J2 Conn_01x02_Male, J3 Conn_01x02_Male, U1 TPS61087DSCR, U2 LM1117-3.3

Commit message: Actualizacion
Parts:
- added REF**: KiCad-Logo2_5mm_SilkScreen, Symbol:KiCad-Logo2_5mm_SilkScreen, F.Cu at (208.8, 111.7)
Other:
- board text added: "Modulo buck-boost v1.0"
